Commit message: adjusted camera angle

File: src/robot_description/urdf/turtlebot3_waffle_pi.urdf (robot description, URDF)
Before this commit: robot turtlebot3_waffle_pi, 11 links, 10 joints
Joints:
- joint camera_rgb_optical_joint: origin xyz=0 0 0 rpy=-1.57 0 -1.57 -> xyz=0 0 0 rpy=-1.57 -1.57 -1.57

Commit message: fixed camera roll

File: src/robot_description/urdf/turtlebot3_waffle_pi.urdf (robot description, URDF)
Before this commit: robot turtlebot3_waffle_pi, 11 links, 10 joints
Joints:
- joint camera_rgb_optical_joint: origin xyz=0 0 0 rpy=-1.57 -1.57 -1.57 -> xyz=0 0 0 rpy=1.57 -1.57 -1.57

Commit message: moved to foxy

File: src/robot_description/urdf/turtlebot3_waffle_pi.urdf (robot description, URDF)
Before this commit: robot turtlebot3_waffle_pi, 11 links, 10 joints
Links:
- link base_link: geometry collision box size=0.266 0.266 0.094; visual mesh filename=package://turtlebot3_description/meshes/bases/waffle_pi_bas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 scale=0.001 0.001 0.001
- link base_scan: geometry collision cylinder length=0.0315 radius=0.055; visual mesh filename=package://turtlebot3_description/meshes/sensors/lds.stl scale=0.001 0.001 0.001
- link wheel_left_link: geometry collision cylinder length=0.018 radius=0.033; visual mesh filename=package://turtlebot3_description/meshes/wheels/left_tire.stl scale=0.001 0.001 0.001
- link wheel_right_link: geometry collision cylinder length=0.018 radius=0.033; visual mesh filename=package://turtlebot3_description/meshes/wheels/right_tire.s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 scale=0.001 0.001 0.001
